File: Sleepy Fox.kicad_pcb (KiCad board)
At the start: 2 copper layers, 273.6 x 102.7 mm, 97 parts, among them SW1 SW_Push, U1 ProMicro

Commit message: updates
big updates for firmware
Other:
- net class Default removed
